Commit message: initialize safety filter

File: src/arm_sim_node/urdf/Arm.urdf (robot description, URDF)
Before this commit: robot Arm, 33 links, 32 joints
Links:
- added link link4_sensor1_camera_gz_link, mass 0.000001
- added link link4_sensor1_tof_gz_link, mass 0.000001
- added link link4_sensor2_camera_gz_link, mass 0.000001
- added link link4_sensor2_tof_gz_link, mass 0.000001
- added link world
Joints:
- added joint link4_sensor1_camera_gz_joint: type fixed, parent link4_sensor1_camera_link, child link4_sensor1_camera_gz_link, origin xyz=0 0 0 rpy=1.5707963267949 -1.5707963267949 0, axis 0 0 0
- added joint link4_sensor1_tof_gz_joint: type fixed, parent link4_sensor1_tof_link, child link4_sensor1_tof_gz_link, origin xyz=0 0 0 rpy=1.5707963267949 -1.5707963267949 0, axis 0 0 0
- added joint link4_sensor2_camera_gz_joint: type fixed, parent link4_sensor2_camera_link, child link4_sensor2_camera_gz_link, origin xyz=0 0 0 rpy=1.5707963267949 -1.5707963267949 0, axis 0 0 0
- added joint link4_sensor2_tof_gz_joint: type fixed, parent link4_sensor2_tof_link, child link4_sensor2_tof_gz_link, origin xyz=0 0 0 rpy=1.5707963267949 -1.5707963267949 0, axis 0 0 0
- added joint world_to_base_fixed_joint: type fixed, parent world, child base_link, origin xyz=0 0 0 rpy=0 0 0
- joint EE_sensor1_camera_joint: origin xyz=-0.0055 -0.0055 0.023 rpy=0 0 0 -> xyz=-0.0055 -0.0055 0.023 rpy=0 0 1.5708
- joint EE_sensor1_tof_joint: origin xyz=0.00549999999907926 0.00550000000001525 0.0229999999747452 rpy=0 0 0 -> xyz=0.0055 0.0055 0.023 rpy=0 0 1.5708
- joint EE_sensor2_camera_joint: origin xyz=-0.00549999999999995 -0.0055 0.0229999999999999 rpy=0 0 0 -> xyz=-0.0055 -0.0055 0.023 rpy=0 0 1.5708
- joint EE_sensor2_tof_joint: origin xyz=0.0055 0.0055 0.0229999999999999 rpy=0 0 0 -> xyz=0.0055 0.0055 0.023 rpy=0 0 1.5708
- joint link2_sensor1_camera_joint: origin xyz=-0.00549999999999967 0.00549999999999994 -0.0569999999999999 rpy=3.14159265358979 0 0 -> xyz=-0.0055 0.0055 -0.057 rpy=-3.1416 0 -1.5708
- joint link2_sensor1_tof_joint: origin xyz=0.00550000000000034 -0.00550000000000006 -0.0569999999999999 rpy=3.14159265358979 0 0 -> xyz=0.0055 -0.0055 -0.057 rpy=-3.1416 0 -1.5708
- joint link2_sensor2_camera_joint: origin xyz=-0.00550000000000012 0.00550000000000011 -0.0569999999999999 rpy=-3.14159265358979 0 0 -> xyz=-0.0055 0.0055 -0.057 rpy=-3.1416 0 -1.5708
- joint link2_sensor2_tof_joint: origin xyz=0.00549999999999984 -0.00549999999999989 -0.0569999999999999 rpy=-3.14159265358979 0 0 -> xyz=0.0055 -0.0055 -0.057 rpy=-3.1416 0 -1.5708
- joint link3_sensor1_camera_joint: origin xyz=0.00549999999999995 0.0055 0.023 rpy=0 0 -3.14159265358979 -> xyz=0.0055 0.0055 0.023 rpy=0 0 -1.5708
- joint link3_sensor1_tof_joint: origin xyz=-0.0055 -0.0055 0.023 rpy=0 0 -3.14159265358979 -> xyz=-0.0055 -0.0055 0.023 rpy=0 0 -1.5708
- joint link3_sensor2_camera_joint: origin xyz=-0.0055 -0.0055 0.023 rpy=0 0 0 -> xyz=-0.0055 -0.0055 0.023 rpy=0 0 1.5708
- joint link3_sensor2_tof_joint: origin xyz=0.0055 0.0055 0.023 rpy=0 0 0 -> xyz=0.0055 0.0055 0.023 rpy=0 0 1.5708
- joint link4_sensor1_camera_joint: origin xyz=0.0055000000000017 0.00550000000000028 0.0230000000000001 rpy=0 0 3.14159265358979 -> xyz=0.0055 0.0055 0.023 rpy=0 0 -1.5708
- joint link4_sensor1_tof_joint: origin xyz=-0.0054999999999983 -0.00549999999999984 0.0230000000000001 rpy=0 0 3.14159265358979 -> xyz=-0.0055 -0.0055 0.023 rpy=0 0 -1.5708
- joint link4_sensor2_camera_joint: origin xyz=-0.00549999999999995 -0.0055 0.023 rpy=0 0 0 -> xyz=-0.0055 -0.0055 0.023 rpy=0 0 1.5708
- joint link4_sensor2_tof_joint: origin xyz=0.00549999999999995 0.0055 0.023 rpy=0 0 0 -> xyz=0.0055 0.0055 0.023 rpy=0 0 1.5708
